File: caddata/am-pcb4/pcb4-28m.kicad_sch (KiCad schematic)
At the start: 237 parts, among them IC51 UTC7642, J101 Univ_03x05, J102 Univ_03x02, J103 Univ_03x05, J104 Univ_04x08, J201 AudioPlug4, J202 AudioPlug4, J91 Conn_Coaxial, J92 Conn_Coaxial, J93 AudioJack4, J94 AudioJack2_Ground, J95 AudioJack3, K201 Y14H-1C-9DS, K91 Y14H-1C-9DS, Q11 BF256B, Q201 2SC1815, Q21 2SC1959, Q31 2SC1959, Q61 2SC1959, Q71 2SC1959, SW201 SW_SPDT_MSM, SW202 SW_Push, T11 7T25, T21 7T25, T31 7T1R0, T41 7S1R0, T42 7S1R0, T61 7T25, T62 7T25, T71 7T25, T91 7T50, U201 Microphone, U41 CF-455, U51 LM386, U71 LM386, U91 Microphone, X21 27.000M, X61 28.375M

Commit message: Add files via upload
Parts:
- R15: value 100 -> 220
- R73: value 22 -> 100
- T41, T42: value 7S1R0 -> 7T1R0
Other:
- note removed: "2M chebyshev 3300p,4.7u,4700p,4.7u,3300p 3M chebyshev 2200p,3.3u,3300p,3.3u,2200p 2M butterworth 1000p,6.8u,3300p,6.8u,1000p 3M butterworth 680p,4.7u,2200p,4.7u,680p"
- note removed: "35M chebyshev 150p,330n,330p,330n,150p 60M chebyshev 82p,150n,120p,150n,82p 35M butterworth 56p,330n,180p,330n,56p 60M butterworth 33p,220n,100p,220n,33p"
- note removed: "50M 7T1R0 300p 1.7M 16.9344*3 -16.384*3 = 1.6512 28M 7T1R0 370p 1.4M 28.375-27.000 = 1.375"
- note removed: "50M 7T50 10p 2SC1923 16.384M x 3 28M 7T25 33p 2SC1959 27.000M"
- note removed: "50M 7T50 12p 2SC1923 16.9344M x 3 28M 7T25 33p 2SC1959 28.375M 7M 7T7 100p 2SC1959 7.181M"
- note removed: "Drill=3.2mm Wire=0.2mm Length=2.54mm r=1.7-1.8 Turn 7 = 136-150n Turn 9 = 226-248n Turn 11 = 338-371n"
- note removed: "Drill=3.2mm Wire=0.4mm Length=5.12mm r=1.8-1.9 Turn 9 = 153-169n Turn 11 = 230-253n Turn 13 = 321-353n"
- note removed: "R73 extremely low power 1k normal about 10mW 22"
Changed lines of the file:
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@@
     (effects (font (size 1.27 1.27)) (justify left bottom))
   )
-  (text "50M 7T1R0 300p 1.7M\n16.9344*3 -16.384*3 = 1.6512\n\n28M 7T1R0 370p 1.4M\n28.375-27.000 = 1.375\n"
-    (at 184.15 158.75 0)
-    (effects (font (size 1.27 1.27)) (justify left bottom))
-  )
   (text "D21\n1SV161\n1T32\n1SV136A" (at 42.545 231.775 0)
     (effects (font (size 1.27 1.27)) (justify left bottom))
@@
     (effects (font (size 1.27 1.27)) (justify left bottom))
   )
-  (text "R73\nextremely low power\n  1k\nnormal about 10mW\n  22\n"
-    (at 254 322.58 0)
-    (effects (font (size 1.27 1.27)) (justify left bottom))
-  )
   (text "Jumper\nTP45-TP55\nIF signal" (at 267.97 60.96 0)
     (effects (font (size 1.27 1.27)) (justify left bottom))
@@
     (effects (font (size 1.27 1.27)) (justify left bottom))
   )
-  (text "Drill=3.2mm Wire=0.4mm\nLength=5.12mm  r=1.8-1.9\nTurn  9 = 153-169n\nTurn 11 = 230-253n\nTurn 13 = 321-353n\n"
-    (at 350.52 248.285 0)
-    (effects (font (size 1.27 1.27)) (justify left bottom))
-  )
-  (text "2M chebyshev\n 3300p,4.7u,4700p,4.7u,3300p\n3M chebyshev\n 2200p,3.3u,3300p,3.3u,2200p\n2M butterworth\n 1000p,6.8u,3300p,6.8u,1000p\n3M butterworth\n 680p,4.7u,2200p,4.7u,680p\n\n"
-    (at 227.965 69.85 0)
-    (effects (font (size 1.27 1.27)) (justify left bottom))
-  )
   (text "RX" (at 180.975 175.26 0)
     (effects (font (size 1.27 1.27)) (justify left bottom))
@@
     (effects (font (size 1.27 1.27)) (justify left bottom))
   )
-  (text "Drill=3.2mm Wire=0.2mm\nLength=2.54mm  r=1.7-1.8\nTurn  7 = 136-150n\nTurn  9 = 226-248n\nTurn 11 = 338-371n\n"
-    (at 320.04 248.285 0)
-    (effects (font (size 1.27 1.27)) (justify left bottom))
-  )
   (text "PTT" (at 127 534.67 0)
     (effects (font (size 1.27 1.27)) (justify left bottom))
@@
     (effects (font (size 1.27 1.27)) (justify left bottom))
   )
-  (text "50M 7T50 12p\n2SC1923\n16.9344M x 3\n\n28M 7T25 33p\n2SC1959\n28.375M \n\n7M 7T7 100p\n2SC1959\n7.181M \n"
-    (at 98.425 364.49 0)
-    (effects (font (size 1.27 1.27)) (justify left bottom))
-  )
   (text "RF Detector for TEST\n(If you have only a tester)" (at 313.055 317.5 0)
     (effects (font (size 1.27 1.27)) (justify left bottom))
@@
     (effects (font (size 1.27 1.27)) (justify left bottom))
   )
-  (text "35M chebyshev\n 150p,330n,330p,330n,150p\n60M chebyshev\n  82p,150n,120p,150n,82p\n35M butterworth\n  56p,330n,180p,330n,56p\n60M butterworth\n  33p,220n,100p,220n,33p\n\n"
-    (at 287.655 252.73 0)
-    (effects (font (size 1.27 1.27)) (justify left bottom))
-  )
-  (text "50M 7T50 10p\n2SC1923\n16.384M x 3\n\n28M 7T25 33p\n2SC1959\n27.000M \n"
-    (at 120.015 204.47 0)
-    (effects (font (size 1.27 1.27)) (justify left bottom))
-  )
   (text "Jumper\nTP51-TP52\nIC's power" (at 357.505 130.81 0)
     (effects (font (size 1.27 1.27)) (justify left bottom))
@@
       (effects (font (size 1.27 1.27)) (justify left))
     )
-    (property "Value" "100" (at 92.71 90.17 0)
+    (property "Value" "220" (at 92.71 90.17 0)
       (effects (font (size 1.27 1.27)) (justify left))
     )
@@
       (effects (font (size 1.27 1.27)) (justify left))
     )
-    (property "Value" "22" (at 257.81 305.435 0)
+    (property "Value" "100" (at 257.81 305.435 0)
       (effects (font (size 1.27 1.27)) (justify left))
     )
@@
       (effects (font (size 1.27 1.27)))
     )
-    (property "Value" "7S1R0" (at 237.49 122.555 0)
+    (property "Value" "7T1R0" (at 237.49 122.555 0)
       (effects (font (size 1.27 1.27)))
     )
@@
       (effects (font (size 1.27 1.27)))
     )
-    (property "Value" "7S1R0" (at 289.56 122.555 0)
+    (property "Value" "7T1R0" (at 289.56 122.555 0)
       (effects (font (size 1.27 1.27)))
     )
